Commit message: Update locobot_description.urdf

File: robots/LoCoBot/locobot_description/urdf/locobot_description.urdf (robot description, URDF)
Before this commit: robot locobot, 25 links, 24 joints
Joints:
- joint cam_mount_joint: origin xyz=-0.03751 0 0.1458 rpy=0 0 0 -> xyz=-0.03751 0 0.1331 rpy=0 0 0

Commit message: updated urdf

File: robots/LoCoBot/locobot_description/urdf/locobot_description.urdf (robot description, URDF)
Before this commit: robot locobot, 25 links, 24 joints
Links:
- link plate_1: geometry collision mesh filename=package://locobot_description/meshes/plate.STL; visual mesh filename=package://locobot_description/meshes/plate.STL
- link plate_2: geometry collision mesh filename=package://locobot_description/meshes/plate.STL; visual mesh filename=package://locobot_description/meshes/plate.STL
Joints:
- joint arm_base_link_joint: origin xyz=0 0 -0.010 rpy=0 0 0 -> xyz=0 0 0.001 rpy=0 0 0
- joint plate_1_joint: origin xyz=0.0973 0 0.095 rpy=0 0 0 -> xyz=0.0973 0 0.0902375 rpy=0 0 0
